File: Touchpad-Spacer.kicad_pcb (KiCad board)
At the start: 2 copper layers, 283.2 x 112.6 mm, 0 parts

Commit message: New version, more subtle & no exposed lead solder
Routing:
- removed copper zone on F.Cu, net (none)
Other:
- board text added: "JLCJLCJLCJLC"
